Commit message: wip: 손 하드웨어 임시 수정 (그리퍼/카메라 STL 부착)
- openarm_hand.xacro: hand visual 을 openarm_gripper_1.STL 로 교체,
  오른팔에 end_point_link (gripper_2.STL) + camera_base_link (Gemini 336.STL) 추가,
  finger 링크/조인트 제거, hand_tcp 는 왼팔 전용으로 변경.
- 새 visual 메시 4종 추가 (openarm_gripper_1/2/full, Gemini 336).
- bimanual.rviz: 시각 확인용 변경.

임시 커밋 — 추후 정리/원복 예정.

File: urdf/ee/openarm_hand.xacro (robot description, xacro)
@@ -8,6 +8,19 @@
       <xacro:property name="ee_prefix" value="openarm_${arm_prefix}" />
     </xacro:unless>
-    <xacro:ee_link_with_sc name="hand" prefix="${ee_prefix}" ee_kinematics_link="${ee_kinematics_link}"/>
-    <!-- <link name="${ee_prefix}hand"/> -->
+    <link name="${ee_prefix}hand">
+      <visual name="${ee_prefix}hand_visual">
+        <xacro:openarm-ee-kinematics-link config="${ee_kinematics_link}" name="hand" />
+        <geometry>
+          <mesh filename="package://${description_pkg}/meshes/ee/${ee_type}/visual/openarm_gripper_1.STL" scale="0.001 0.001 0.001" />
+        </geometry>
+      </visual>
+      <collision name="${ee_prefix}hand_collision">
+        <xacro:openarm-ee-kinematics-link config="${ee_kinematics_link}" name="hand" />
+        <geometry>
+          <mesh filename="package://${description_pkg}/meshes/ee/${ee_type}/collision/hand.stl" scale="0.001 0.001 0.001" />
+        </geometry>
+      </collision>
+      <xacro:ee-inertials name="hand" />
+    </link>
     <xacro:unless value="${connected_to == ''}">
       <!-- <joint name="${ee_prefix}hand_joint" type="fixed"> -->
@@ -18,55 +31,42 @@
       </joint>
     </xacro:unless>
-    <!-- Define the hand_tcp frame -->
-    <link name="${ee_prefix}hand_tcp" />
-    <joint name="${ee_prefix}hand_tcp_joint" type="fixed">
-      <origin xyz="${tcp_xyz}" rpy="${tcp_rpy}" />
-      <parent link="${ee_prefix}hand" />
-      <child link="${ee_prefix}hand_tcp" />
-    </joint>
-    <link name="${ee_prefix}left_finger">
-      <visual name="${ee_prefix}left_finger_visual">
-        <xacro:openarm-ee-kinematics-link config="${ee_kinematics_link}" name="left_finger" />
+    <!-- hand_tcp: left arm only (right arm uses end_point_link instead) -->
+    <xacro:unless value="${arm_prefix == 'right_'}">
+      <link name="${ee_prefix}hand_tcp" />
+      <joint name="${ee_prefix}hand_tcp_joint" type="fixed">
+        <origin xyz="${tcp_xyz}" rpy="${tcp_rpy}" />
+        <parent link="${ee_prefix}hand" />
+        <child link="${ee_prefix}hand_tcp" />
+      </joint>
+    </xacro:unless>
+    <!-- IK 기준 프레임 (오른팔 전용): 그리퍼 끝단 -->
+    <xacro:if value="${arm_prefix == 'right_'}">
+      <link name="end_point_link">
+        <visual name="end_point_link_visual">
+          <origin xyz="0 0 0" rpy="0 0 0" />
+          <geometry>
+            <mesh filename="package://${description_pkg}/meshes/ee/${ee_type}/visual/openarm_gripper_2.STL" scale="0.001 0.001 0.001" />
+          </geometry>
+        </visual>
+      </link>
+      <joint name="end_point_link_joint" type="fixed">
+        <origin xyz="0.015001 0 0.1275005" rpy="0 0 0" />
+        <parent link="${ee_prefix}hand" />
+        <child link="end_point_link" />
+      </joint>
+    </xacro:if>
+    <!-- Gemini 336 카메라 베이스 (양쪽 공통) -->
+    <link name="${ee_prefix}camera_base_link">
+      <visual name="${ee_prefix}camera_base_link_visual">
+        <origin xyz="0 0 0" rpy="0 0 0" />
         <geometry>
-          <mesh filename="package://${description_pkg}/meshes/ee/${ee_type}/visual/finger.dae" scale="0.001 0.001 0.001"/>
+          <mesh filename="package://${description_pkg}/meshes/ee/${ee_type}/visual/Gemini 336.STL" scale="0.001 0.001 0.001" />
         </geometry>
       </visual>
-      <collision name="${ee_prefix}left_finger_collision">
-        <xacro:openarm-ee-kinematics-link config="${ee_kinematics_link}" name="left_finger" />
-        <geometry>
-          <mesh filename="package://${description_pkg}/meshes/ee/${ee_type}/collision/finger.stl" scale="0.001 0.001 0.001" />
-        </geometry>
-      </collision>
-      <xacro:ee-inertials name="left_finger"/>
     </link>
-    <link name="${ee_prefix}right_finger">
-      <visual name="${ee_prefix}right_finger_visual">
-        <xacro:openarm-ee-kinematics-link config="${ee_kinematics_link}" name="right_finger" />
-        <geometry>
-          <mesh filename="package://${description_pkg}/meshes/ee/${ee_type}/visual/finger.dae" scale="0.001 -0.001 0.001"/>
-        </geometry>
-      </visual>
-      <collision name="${ee_prefix}right_finger_collision">
-        <xacro:openarm-ee-kinematics-link config="${ee_kinematics_link}" name="right_finger" />
-        <geometry>
-          <mesh filename="package://${description_pkg}/meshes/ee/${ee_type}/collision/finger.stl" scale="0.001 -0.001 0.001" />
-        </geometry>
-      </collision>
-      <xacro:ee-inertials name="right_finger"/>
-    </link>
-    <joint name="${ee_prefix}finger_joint1" type="prismatic">
+    <joint name="${ee_prefix}camera_base_link_joint" type="fixed">
+      <origin xyz="-0.017999 0 0.0364005" rpy="0 0 0" />
       <parent link="${ee_prefix}hand" />
-      <child link="${ee_prefix}right_finger" />
-      <origin xyz="0 -0.006 0.015" rpy="0 0 0" />
-      <axis xyz="0 -1 0" />
-      <limit effort="333" lower="0.0" upper="0.044" velocity="10.0" />
-    </joint>
-    <joint name="${ee_prefix}finger_joint2" type="prismatic">
-      <parent link="${ee_prefix}hand" />
-      <child link="${ee_prefix}left_finger" />
-      <origin xyz="0 0.006 0.015" rpy="0 0 0" />
-      <axis xyz="0 1 0" />
-      <limit effort="333" lower="0.0" upper="0.044" velocity="10.0" />
-      <mimic joint="${ee_prefix}finger_joint1" />
+      <child link="${ee_prefix}camera_base_link" />
     </joint>
   </xacro:macro>
