Commit message: feat: 커스텀 EE(분해형 그리퍼) 지원 추가
- openarm_hand.xacro 에 hand 인자(default false) 분기 추가:
  hand=true 는 기존 통짜 그리퍼(finger joint 포함),
  hand=false 는 base_link / end_point_link / hand_eye_camera 로
  분해된 커스텀 EE 를 부착.
- 커스텀 EE 용 base_link / end_point_link / hand_eye_camera_link STL 추가.
- openarm_robot.xacro: hand 인자를 매크로로 전달하고, ee_type 이
  openarm_hand 이면 hand 값에 관계없이 EE 를 부착하도록 정리.
- v10.urdf.xacro 의 hand 기본값을 false 로 변경.
- kinematics_link.yaml: 분해 모델 기준에 맞춰 hand offset 재캘리브레이션,
  사용하지 않는 left/right_finger 오프셋은 0 으로 리셋.

Co-Authored-By: Claude Opus 4.7 (1M context) <noreply@anthropic.com>

File: urdf/ee/openarm_hand.xacro (robot description, xacro)
@@ -2,5 +2,5 @@
 <robot xmlns:xacro="http://www.ros.org/wiki/xacro" name="hand">
   <!-- safety_distance: Minimum safety distance in [m] by which the collision volumes are expanded and which is enforced during robot motions -->
-  <xacro:macro name="openarm_hand" params="connected_to:='' arm_type arm_prefix:='' ee_type ee_inertials ee_kinematics_link rpy_ee:='0 0 0' xyz_ee:='0 0 0' tcp_xyz:='0 0 0' tcp_rpy:='0 0 0' description_pkg:=openarm_description">
+  <xacro:macro name="openarm_hand" params="connected_to:='' arm_type arm_prefix:='' ee_type ee_inertials ee_kinematics_link rpy_ee:='0 0 0' xyz_ee:='0 0 0' tcp_xyz:='0 0 0' tcp_rpy:='0 0 0' description_pkg:=openarm_description hand:='false'">
     <xacro:property name="ee_prefix" default=""/>
     <xacro:unless value="${arm_type == ''}">
@@ -8,29 +8,17 @@
       <xacro:property name="ee_prefix" value="openarm_${arm_prefix}" />
     </xacro:unless>
-    <link name="${ee_prefix}hand">
-      <visual name="${ee_prefix}hand_visual">
-        <xacro:openarm-ee-kinematics-link config="${ee_kinematics_link}" name="hand" />
-        <geometry>
-          <mesh filename="package://${description_pkg}/meshes/ee/${ee_type}/visual/openarm_gripper_1.STL" scale="0.001 0.001 0.001" />
-        </geometry>
-      </visual>
-      <collision name="${ee_prefix}hand_collision">
-        <xacro:openarm-ee-kinematics-link config="${ee_kinematics_link}" name="hand" />
-        <geometry>
-          <mesh filename="package://${description_pkg}/meshes/ee/${ee_type}/collision/hand.stl" scale="0.001 0.001 0.001" />
-        </geometry>
-      </collision>
-      <xacro:ee-inertials name="hand" />
-    </link>
-    <xacro:unless value="${connected_to == ''}">
-      <!-- <joint name="${ee_prefix}hand_joint" type="fixed"> -->
-      <joint name="${arm_prefix}openarm_hand_joint" type="fixed">
-        <parent link="${connected_to}" />
-        <child link="${ee_prefix}hand" />
-        <origin xyz="${xyz_ee}" rpy="${rpy_ee}" />
-      </joint>
-    </xacro:unless>
-    <!-- hand_tcp: left arm only (right arm uses end_point_link instead) -->
-    <xacro:unless value="${arm_prefix == 'right_'}">
+    <!-- ============================================================== -->
+    <!-- hand=true: 원본 그리퍼 (finger joints 포함)                       -->
+    <!-- ============================================================== -->
+    <xacro:if value="${hand}">
+      <xacro:ee_link_with_sc name="hand" prefix="${ee_prefix}" ee_kinematics_link="${ee_kinematics_link}"/>
+      <xacro:unless value="${connected_to == ''}">
+        <joint name="${arm_prefix}openarm_hand_joint" type="fixed">
+          <parent link="${connected_to}" />
+          <child link="${ee_prefix}hand" />
+          <origin xyz="${xyz_ee}" rpy="${rpy_ee}" />
+        </joint>
+      </xacro:unless>
+      <!-- hand_tcp (양쪽 공통) -->
       <link name="${ee_prefix}hand_tcp" />
       <joint name="${ee_prefix}hand_tcp_joint" type="fixed">
@@ -39,35 +27,147 @@
         <child link="${ee_prefix}hand_tcp" />
       </joint>
-    </xacro:unless>
-    <!-- IK 기준 프레임 (오른팔 전용): 그리퍼 끝단 -->
-    <xacro:if value="${arm_prefix == 'right_'}">
-      <link name="end_point_link">
-        <visual name="end_point_link_visual">
+      <link name="${ee_prefix}left_finger">
+        <visual name="${ee_prefix}left_finger_visual">
+          <xacro:openarm-ee-kinematics-link config="${ee_kinematics_link}" name="left_finger" />
+          <geometry>
+            <mesh filename="package://${description_pkg}/meshes/ee/${ee_type}/visual/finger.dae" scale="0.001 0.001 0.001"/>
+          </geometry>
+        </visual>
+        <collision name="${ee_prefix}left_finger_collision">
+          <xacro:openarm-ee-kinematics-link config="${ee_kinematics_link}" name="left_finger" />
+          <geometry>
+            <mesh filename="package://${description_pkg}/meshes/ee/${ee_type}/collision/finger.stl" scale="0.001 0.001 0.001" />
+          </geometry>
+        </collision>
+        <xacro:ee-inertials name="left_finger"/>
+      </link>
+      <link name="${ee_prefix}right_finger">
+        <visual name="${ee_prefix}right_finger_visual">
+          <xacro:openarm-ee-kinematics-link config="${ee_kinematics_link}" name="right_finger" />
+          <geometry>
+            <mesh filename="package://${description_pkg}/meshes/ee/${ee_type}/visual/finger.dae" scale="0.001 -0.001 0.001"/>
+          </geometry>
+        </visual>
+        <collision name="${ee_prefix}right_finger_collision">
+          <xacro:openarm-ee-kinematics-link config="${ee_kinematics_link}" name="right_finger" />
+          <geometry>
+            <mesh filename="package://${description_pkg}/meshes/ee/${ee_type}/collision/finger.stl" scale="0.001 -0.001 0.001" />
+          </geometry>
+        </collision>
+        <xacro:ee-inertials name="right_finger"/>
+      </link>
+      <joint name="${ee_prefix}finger_joint1" type="prismatic">
+        <parent link="${ee_prefix}hand" />
+        <child link="${ee_prefix}right_finger" />
+        <origin xyz="0 -0.006 0.015" rpy="0 0 0" />
+        <axis xyz="0 -1 0" />
+        <limit effort="333" lower="0.0" upper="0.044" velocity="10.0" />
+      </joint>
+      <joint name="${ee_prefix}finger_joint2" type="prismatic">
+        <parent link="${ee_prefix}hand" />
+        <child link="${ee_prefix}left_finger" />
+        <origin xyz="0 0.006 0.015" rpy="0 0 0" />
+        <axis xyz="0 1 0" />
+        <limit effort="333" lower="0.0" upper="0.044" velocity="10.0" />
+        <mimic joint="${ee_prefix}finger_joint1" />
+      </joint>
+    </xacro:if>
+    <!-- ============================================================== -->
+    <!-- hand=false: 커스텀 EE (base_link / end_point_link / camera 분해)  -->
+    <!-- 오른팔 전용 워크플로 — 왼팔 가드/hand_tcp 없음                      -->
+    <!-- ============================================================== -->
+    <xacro:unless value="${hand}">
+      <!-- 소스 base_link 역할: 그리퍼 베이스.
+           분해 모델(base/end_point/camera)은 소스 URDF 의 joint origin 으로
+           상대 위치가 정의되므로, 통짜 STL 시절 calibrate 된
+           kinematics_link.yaml 의 hand offset 은 적용하지 않는다. -->
+      <link name="${ee_prefix}hand">
+        <visual name="${ee_prefix}hand_visual">
           <origin xyz="0 0 0" rpy="0 0 0" />
           <geometry>
-            <mesh filename="package://${description_pkg}/meshes/ee/${ee_type}/visual/openarm_gripper_2.STL" scale="0.001 0.001 0.001" />
+            <mesh filename="package://${description_pkg}/meshes/ee/${ee_type}/visual/base_link.STL" />
           </geometry>
+          <material name="${ee_prefix}hand_material">
+            <color rgba="0.498039215686275 0.498039215686275 0.498039215686275 1" />
+          </material>
         </visual>
+        <collision name="${ee_prefix}hand_collision">
+          <origin xyz="0 0 0" rpy="0 0 0" />
+          <geometry>
+            <mesh filename="package://${description_pkg}/meshes/ee/${ee_type}/visual/base_link.STL" />
+          </geometry>
+        </collision>
+        <xacro:ee-inertials name="hand" />
+      </link>
+      <xacro:unless value="${connected_to == ''}">
+        <joint name="${arm_prefix}openarm_hand_joint" type="fixed">
+          <parent link="${connected_to}" />
+          <child link="${ee_prefix}hand" />
+          <origin xyz="${xyz_ee}" rpy="${rpy_ee}" />
+        </joint>
+      </xacro:unless>
+      <!-- IK 기준 프레임 / 그리퍼 끝단 -->
+      <link name="end_point_link">
+        <inertial>
+          <origin xyz="-1.23028670139052E-09 1.73472347597681E-18 0.0648443771008311" rpy="0 0 0" />
+          <mass value="0.0534321538206244" />
+          <inertia
+            ixx="4.79644094134221E-05" ixy="-5.32360812357627E-11" ixz="-2.26763003040317E-12"
+            iyy="4.81762945680171E-05" iyz="3.59695627016764E-22"
+            izz="4.57906580222582E-06" />
+        </inertial>
+        <visual>
+          <origin xyz="0 0 0" rpy="0 0 0" />
+          <geometry>
+            <mesh filename="package://${description_pkg}/meshes/ee/${ee_type}/visual/end_point_link.STL" />
+          </geometry>
+          <material name="end_point_link_material">
+            <color rgba="0.498039215686275 0.498039215686275 0.498039215686275 1" />
+          </material>
+        </visual>
+        <collision>
+          <origin xyz="0 0 0" rpy="0 0 0" />
+          <geometry>
+            <mesh filename="package://${description_pkg}/meshes/ee/${ee_type}/visual/end_point_link.STL" />
+          </geometry>
+        </collision>
       </link>
       <joint name="end_point_link_joint" type="fixed">
-        <origin xyz="0.015001 0 0.1275005" rpy="0 0 0" />
+        <origin xyz="0.0155 0 0.1275" rpy="${pi} 0 ${pi/2}" />
         <parent link="${ee_prefix}hand" />
         <child link="end_point_link" />
       </joint>
-    </xacro:if>
-    <!-- Gemini 336 카메라 베이스 (양쪽 공통) -->
-    <link name="${ee_prefix}camera_base_link">
-      <visual name="${ee_prefix}camera_base_link_visual">
-        <origin xyz="0 0 0" rpy="0 0 0" />
-        <geometry>
-          <mesh filename="package://${description_pkg}/meshes/ee/${ee_type}/visual/Gemini 336.STL" scale="0.001 0.001 0.001" />
-        </geometry>
-      </visual>
-    </link>
-    <joint name="${ee_prefix}camera_base_link_joint" type="fixed">
-      <origin xyz="-0.017999 0 0.0364005" rpy="0 0 0" />
-      <parent link="${ee_prefix}hand" />
-      <child link="${ee_prefix}camera_base_link" />
-    </joint>
+      <!-- Gemini 336 hand-eye 카메라 베이스 -->
+      <link name="end_effector_camera_base_link">
+        <inertial>
+          <origin xyz="0.00503091354265199 6.13311072507168E-06 0.0123843639611123" rpy="0 0 0" />
+          <mass value="0.0197150970342339" />
+          <inertia
+            ixx="1.4476965753632E-05"  ixy="-6.23479322830121E-09" ixz="-1.1580268544267E-08"
+            iyy="2.80948348806754E-06" iyz="-1.00940904623301E-08"
+            izz="1.4833122948371E-05" />
+        </inertial>
+        <visual>
+          <origin xyz="0 0 0" rpy="0 0 0" />
+          <geometry>
+            <mesh filename="package://${description_pkg}/meshes/ee/${ee_type}/visual/hand_eye_camera_link.STL" />
+          </geometry>
+          <material name="end_effector_camera_base_link_material">
+            <color rgba="0.792156862745098 0.819607843137255 0.933333333333333 1" />
+          </material>
+        </visual>
+        <collision>
+          <origin xyz="0 0 0" rpy="0 0 0" />
+          <geometry>
+            <mesh filename="package://${description_pkg}/meshes/ee/${ee_type}/visual/hand_eye_camera_link.STL" />
+          </geometry>
+        </collision>
+      </link>
+      <joint name="end_effector_camera_base_link_joint" type="fixed">
+        <origin xyz="-0.0425 0 0.036401" rpy="${pi} ${-pi/2} 0" />
+        <parent link="${ee_prefix}hand" />
+        <child link="end_effector_camera_base_link" />
+      </joint>
+    </xacro:unless>
   </xacro:macro>
 </robot>

File: urdf/robot/openarm_robot.xacro (robot description, xacro)
@@ -138,5 +138,5 @@
             </xacro:if>
         </xacro:if>
-        <xacro:if value="$(eval hand and ee_type == 'openarm_hand')">
+        <xacro:if value="${ee_type == 'openarm_hand'}">
             <xacro:if value="${include_left}">
                 <xacro:openarm_hand
@@ -152,4 +152,5 @@
                     tcp_rpy="$(arg tcp_rpy)"
                     description_pkg="$(arg description_pkg)"
+                    hand="${hand}"
                 />
             </xacro:if>
@@ -167,4 +168,5 @@
                     tcp_rpy="$(arg tcp_rpy)"
                     description_pkg="$(arg description_pkg)"
+                    hand="${hand}"
                 />
             </xacro:if>
@@ -196,9 +198,8 @@
             can_fd="${can_fd}"/>
         </xacro:if>
-        <xacro:if value="${hand and ee_type == 'openarm_hand'}">
+        <xacro:if value="${ee_type == 'openarm_hand'}">
         <xacro:property name="special_connection" value="$(arg special_connection)" />
         <!-- <xacro:property name="connection" value="${special_connection if special_connection != '' else arm_type + '_link7'}" /> -->
         <xacro:property name="connection" value="${special_connection if special_connection != '' else 'openarm' + '_link7'}" />
-        <xacro:if value="$(eval hand and ee_type == 'openarm_hand')">
         <xacro:openarm_hand
             connected_to="${arm_prefix_modified}${connection}"
@@ -212,6 +213,6 @@
             tcp_xyz="$(arg tcp_xyz)"
             tcp_rpy="$(arg tcp_rpy)"
-            description_pkg="$(arg description_pkg)"/>
-        </xacro:if>
+            description_pkg="$(arg description_pkg)"
+            hand="${hand}"/>
         </xacro:if>
         </xacro:if>

File: urdf/robot/v10.urdf.xacro (robot description, xacro)
@@ -6,5 +6,5 @@
   <xacro:arg name="ee_type" default="openarm_hand" />
   <xacro:arg name="no_prefix" default="false"/>
-  <xacro:arg name="hand" default="true" />
+  <xacro:arg name="hand" default="false" />
   <xacro:if value="$(eval ee_type == 'none')">
     <xacro:property name="hand" value="false"/>
